File: Sensing.kicad_pcb (KiCad board)
At the start: 2 copper layers, 655.9 x 20 mm, 86 parts, among them IC1 LM358BIDDFR, IC10 H11L1SM, IC11 LM358BIDDFR, IC12 H11L1SM, IC2 H11L1SM, IC3 LM358BIDDFR, IC4 H11L1SM, IC5 LM358BIDDFR, IC6 H11L1SM, IC7 LM358BIDDFR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

Commit message: added shorter connector
Parts:
- J1: footprint Connector_Hirose:Hirose_DF11-16DP-2DSA_2x08_P2.00mm_Vertical -> KiCad:117347426
- moved J1 2.25 mm to (660.4, 29.6), turned to 180 degrees
Connections:
- J1 pad 1: V12 -> V2
- J1 pad 10: V4 -> V10
- J1 pad 11: V3 -> V11
- J1 pad 12: GND -> +5V
- J1 pad 13: V2 -> THERMO
- J1 pad 14: +5V -> GND
- J1 pad 15: THERMO -> V12
- J1 pad 16: V1 -> V13
- J1 pad 2: V13 -> V1
- J1 pad 3: V11 -> V3
- J1 pad 4: V10 -> V4
- J1 pad 5: V9 -> V5
- J1 pad 6: V8 -> V6
- J1 pad 8: V6 -> V8
- J1 pad 9: V5 -> V9
Routing:
- net THERMO: track 648.4 -> 634.8 mm
- net +5V: track 648.8 -> 635.9 mm
- net GND: track 655.1 -> 643.3 mm
- net V1: track 665.8 -> 656.8 mm, vias 3 -> 4
- net V2: track 632.0 -> 626.0 mm, vias 2 -> 3
- net V3: track 549.7 -> 544.7 mm, vias 3 -> 4
- net V5: track 442.3 -> 438.2 mm, vias 3 -> 4
- net V4: track 540.0 -> 535.9 mm, vias 2 -> 3
- net V7: track 338.9 -> 335.7 mm, vias 3 -> 4
- net V6: track 434.2 -> 431.1 mm, vias 2 -> 3
- net V9: track 238.8 -> 236.6 mm, vias 3 -> 4
- net V8: track 328.5 -> 326.3 mm, vias 2 -> 3
- net V10: track 224.7 -> 223.5 mm, vias 2 -> 3
- net V11: track 132.4 -> 131.3 mm, vias 3 -> 4
- net V12: track 116.7 -> 117.6 mm
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